Commit message: modified ergo data

File: software/poppy_ergo_jr/poppy_ergo_jr.urdf (robot description, URDF)
Before this commit: robot PoppyErgoJr, 7 links, 6 joints
Links:
- link section_4: geometry collision mesh filename=package://PoppyErgoJr/meshes/holder_section.STL; visual mesh filename=package://PoppyErgoJr/meshes/holder_section.STL
- link tip: geometry collision mesh filename=package://PoppyErgoJr/meshes/holder_visual.STL; visual mesh filename=package://PoppyErgoJr/meshes/holder_visual.STL

Commit message: holder urdf

File: software/poppy_ergo_jr/poppy_ergo_jr.urdf (robot description, URDF)
Before this commit: robot PoppyErgoJr, 7 links, 6 joints
Links:
- link tip: geometry collision mesh filename=package://PoppyErgoJr/meshes/holder.STL; visual mesh filename=package://PoppyErgoJr/meshes/holder.STL

Commit message: poppyholder urdf

File: software/poppy_ergo_jr/poppy_ergo_jr.urdf (robot description, URDF)
Before this commit: robot PoppyErgoJr, 7 links, 6 joints
Links:
- removed link section_4
- removed link tip
- added link holder, mass 0.00493222432428107; collision mesh filename=package://PoppyErgoJr_holder/meshes/holder.STL; visual mesh filename=package://PoppyErgoJr_holder/meshes/holder.STL
- added link holder_section, mass 0.0387960284371531; collision mesh filename=package://PoppyErgoJr_holder/meshes/holder_section.STL; visual mesh filename=package://PoppyErgoJr_holder/meshes/holder_section.STL
- link base_link: mass 0.0802410895423366 -> 0.0802410895423482; geometry collision mesh filename=package://PoppyErgoJr_holder/meshes/base_link.STL; visual mesh filename=package://PoppyErgoJr_holder/meshes/base_link.STL
- link long_U: geometry collision mesh filename=package://PoppyErgoJr_holder/meshes/long_U.STL; visual mesh filename=package://PoppyErgoJr_holder/meshes/long_U.STL
- link section_1: mass 0.0201321844066136 -> 0.0201321844066143; geometry collision mesh filename=package://PoppyErgoJr_holder/meshes/section_1.STL; visual mesh filename=package://PoppyErgoJr_holder/meshes/section_1.STL
- link section_2: mass 0.017821725151696 -> 0.0178217251516966; geometry collision mesh filename=package://PoppyErgoJr_holder/meshes/section_2.STL; visual mesh filename=package://PoppyErgoJr_holder/meshes/section_2.STL
- link section_3: mass 0.0201321844066136 -> 0.0201321844066143; geometry collision mesh filename=package://PoppyErgoJr_holder/meshes/section_3.STL; visual mesh filename=package://PoppyErgoJr_holder/meshes/section_3.STL
Joints:
- joint m5: child section_4 -> holder_section; origin xyz=0 -0.0151782258778753 -0.048 rpy=-1.5707963267949 0 0 -> xyz=0 -0.0151782258778752 -0.048 rpy=-3.14159265358979 0 0
- joint m6: axis 0 -1 0 -> 0 0 -1; child tip -> holder; origin xyz=0 0.054 0 rpy=1.5707963267949 1.5707963267949 0 -> xyz=0 0 0.0579999999999998 rpy=1.5707963267949 3.4690027011428E-32 3.14159265358979; parent section_4 -> holder_section

Commit message: mesh update to PoppyErgoJr

File: software/poppy_ergo_jr/poppy_ergo_jr.urdf (robot description, URDF)
Before this commit: robot PoppyErgoJr, 7 links, 6 joints
Links:
- link base_link: geometry collision mesh filename=package://PoppyErgoJr/meshes/base_link.STL; visual mesh filename=package://PoppyErgoJr/meshes/base_link.STL
- link holder: geometry collision mesh filename=package://PoppyErgoJr/meshes/holder.STL; visual mesh filename=package://PoppyErgoJr/meshes/holder.STL
- link holder_section: geometry collision mesh filename=package://PoppyErgoJr/meshes/holder_section.STL; visual mesh filename=package://PoppyErgoJr/meshes/holder_section.STL
- link long_U: geometry collision mesh filename=package://PoppyErgoJr/meshes/long_U.STL; visual mesh filename=package://PoppyErgoJr/meshes/long_U.STL
- link section_1: geometry collision mesh filename=package://PoppyErgoJr/meshes/section_1.STL; visual mesh filename=package://PoppyErgoJr/meshes/section_1.STL
- link section_2: geometry collision mesh filename=package://PoppyErgoJr/meshes/section_2.STL; visual mesh filename=package://PoppyErgoJr/meshes/section_2.STL
- link section_3: geometry collision mesh filename=package://PoppyErgoJr/meshes/section_3.STL; visual mesh filename=package://PoppyErgoJr/meshes/section_3.STL
